File: cyborg_ring_v0.sch (EAGLE design)
At the start: 0 parts

Commit message: Schematic
Parts:
- added C1: 100n, rcl:C-EUC0402K
- added GND, MISO, MOSI, RST, SCK, VCC: TPTP20R, testpad:TPTP20R
- added LED_CON1, LED_CON10, LED_CON11, LED_CON12, LED_CON13, LED_CON14, LED_CON15, LED_CON16, LED_CON2, LED_CON3, LED_CON4, LED_CON5, LED_CON6, LED_CON7, LED_CON8, LED_CON9: R0508-1/2, cyborg_ring:R0508-1/2
- added RCON1, RCON10, RCON11, RCON12, RCON13, RCON14, RCON2, RCON3, RCON4, RCON5, RCON6, RCON7, RCON8, RCON9: R0805-1/2, cyborg_ring:R0805-1/2
- added SW1: (no value), cyborg_ring:SWITCH_PUSHBUTTONC&K_KSS
- added U$1, U$2: BAT+, cyborg_ring:BAT+
- added U$3, U$4: BAT-, cyborg_ring:BAT-
- added U1: ATTINYX5V-LEFT, cyborg_ring:ATTINYX5V-LEFT
- added U2: ATTINYX5V-RIGHT, cyborg_ring:ATTINYX5V-RIGHT
Connections:
- new net GND: C1.2, GND.TP, RCON11.P$1, RCON13.P$1, RCON3.P$1, RCON5.P$1, RCON7.P$1, RCON9.P$1, SW1.P$2, U$4.-
- new net GND1: RCON10.P$1, RCON12.P$1, RCON14.P$1, RCON4.P$1, RCON6.P$1, RCON8.P$1
- new net LEDL_L1: MOSI.TP
- new net LED_L0: LED_CON1.P$1, LED_CON3.P$1, LED_CON5.P$1, LED_CON7.P$1, SCK.TP, U1.PB2
- new net LED_L1: LED_CON11.P$1, LED_CON13.P$1, LED_CON15.P$1, LED_CON9.P$1, U1.PB0
- new net LED_R0: LED_CON14.P$1, LED_CON16.P$1, LED_CON2.P$1, LED_CON4.P$1, U2.PB3
- new net LED_R1: LED_CON10.P$1, LED_CON12.P$1, LED_CON6.P$1, LED_CON8.P$1, U2.PB4
- new net N$11: U$2.+, U$3.-
- new net RST: RCON1.P$1, RST.TP
- new net RST1: RCON2.P$1, U2.PB5
- new net SWITCH: MISO.TP, SW1.P$1, U1.PB1
- new net VCC: C1.1, U$1.+, U1.VCC, VCC.TP
Other:
- note added: "Pad connected to GND"
